File: KOSMOPSU2.sch (KiCad schematic (older format))
At the start: 23 parts, among them J1 Conn_01x03_Male, J2 Conn_02x05_Odd_Even, J3 Conn_01x03_Male, T1 Transformer_1P_2S, U1 L7812, U2 L7912

Commit message: autosync
Parts:
- T1: value Transformer_1P_2S -> Myrra 44440 Transformer 240V
Changed lines of the file:
@@
 P 2650 3200
 F 0 "T1" H 2650 3781 50  0000 C CNN
-F 1 "Transformer_1P_2S" H 2650 3690 50  0000 C CNN
+F 1 "Myrra 44440 Transformer 240V " H 2650 3690 50  0000 C CNN
 F 2 "ROBSLIBRARY:Transformer_Myrra_44440" H 2650 3200 50  0001 C CNN
 F 3 "http://www.farnell.com/datasheets/41284.pdf?_ga=2.233493723.43114568.1597566821-2139994514.1588603417&_gac=1.224077545.1594630648.CjwKCAjwjLD4BRAiEiwAg5NBFqP5waZEob4rUPHshlY-hISIfMy5NeT4Vqv-v37p_oVo35PK2Ko7nhoCuOoQAvD_BwE" H 2650 3200 50  0001 C CNN

Commit message: Fuse Schematic Update
Parts:
- added H2, H3, H4, H5: MountingHole_Pad, MountingHole:MountingHole_2.7mm_M2.5_DIN965_Pad, symbol Mechanical:MountingHole_Pad
- F2, F3: footprint ROBSLIBRARY:googiefuse -> AA-ROB:PCB-20MM-FUSE-HOLDER
Connections:
- net Earth: now also H2.1, H3.1, H4.1, H5.1
Other:
- note added: "Version V0.1.1"
- moved on the sheet: C1, C2, C3, C4, C5, C6, D1, D2, D3, D4, D5, F1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

Commit message: C6 Footprint
Parts:
- C6: footprint Capacitor_THT:CP_Radial_D16.0mm_P7.50mm -> Capacitor_THT:CP_Radial_D6.3mm_P2.50mm
Changed lines of the file:
@@
 F 0 "C6" H 8250 5150 50  0000 L CNN
 F 1 "1uf 50V" V 8100 5150 50  0000 L CNN
-F 2 "Capacitor_THT:CP_Radial_D16.0mm_P7.50mm" H 8288 5150 50  0001 C CNN
+F 2 "Capacitor_THT:CP_Radial_D6.3mm_P2.50mm" H 8288 5150 50  0001 C CNN
 F 3 "~" H 8250 5300 50  0001 C CNN
 	1    8250 5300

Commit message: Value Tidy
Parts:
- F1: value Fuse -> 0.2A 240V
- F2, F3: value Fuse -> 1.5A 240V
Changed lines of the file:
@@
 P 7200 4450
 F 0 "F3" V 7003 4450 50  0000 C CNN
-F 1 "Fuse" V 7094 4450 50  0000 C CNN
+F 1 "1.5A 240V" V 7094 4450 50  0000 C CNN
 F 2 "AA-ROB:PCB-20MM-FUSE-HOLDER" V 7130 4450 50  0001 C CNN
 F 3 "~" H 7200 4450 50  0001 C CNN
@@
 P 7100 5750
 F 0 "F2" V 6903 5750 50  0000 C CNN
-F 1 "Fuse" V 6994 5750 50  0000 C CNN
+F 1 "1.5A 240V" V 6994 5750 50  0000 C CNN
 F 2 "AA-ROB:PCB-20MM-FUSE-HOLDER" V 7030 5750 50  0001 C CNN
 F 3 "~" H 7100 5750 50  0001 C CNN
@@
 U 1 1 5F394CB5
 P 4750 5350
-F 0 "F1" V 4553 5350 50  0000 C CNN
-F 1 "Fuse" V 4644 5350 50  0000 C CNN
+F 0 "F1" V 4650 5350 50  0000 C CNN
+F 1 "0.2A 240V" V 4850 5400 50  0000 C CNN
 F 2 "ROBSLIBRARY:googiefuse" V 4680 5350 50  0001 C CNN
 F 3 "~" H 4750 5350 50  0001 C CNN

Commit message: Cap Update
Parts:
- C3: value .33uf 50V -> .2uf 50V
- C4: value 2uf 50V -> .2uf 50V
- C6: value 1uf 50V -> .1uf 50V
- T1: value Myrra 44440 Transformer 240V -> Myrra 44441 Transformer 240V
Other:
- note added: "Version V0.1.2"
- note removed: "Version V0.1.1"
Changed lines of the file:
@@
 P 5300 5150
 F 0 "T1" H 5300 5731 50  0000 C CNN
-F 1 "Myrra 44440 Transformer 240V " H 5300 5640 50  0000 C CNN
+F 1 "Myrra 44441 Transformer 240V " H 5300 5640 50  0000 C CNN
 F 2 "ROBSLIBRARY:Transformer_Myrra_44440" H 5300 5150 50  0001 C CNN
 F 3 "http://www.farnell.com/datasheets/41284.pdf?_ga=2.233493723.43114568.1597566821-2139994514.1588603417&_gac=1.224077545.1594630648.CjwKCAjwjLD4BRAiEiwAg5NBFqP5waZEob4rUPHshlY-hISIfMy5NeT4Vqv-v37p_oVo35PK2Ko7nhoCuOoQAvD_BwE" H 5300 5150 50  0001 C CNN
@@
 P 7650 4800
 F 0 "C3" H 7850 4800 50  0000 L CNN
-F 1 ".33uf 50V" V 7800 4550 50  0000 L CNN
+F 1 ".2uf 50V" V 7800 4550 50  0000 L CNN
 F 2 "Capacitor_THT:CP_Radial_D6.3mm_P2.50mm" H 7688 4650 50  0001 C CNN
 F 3 "~" H 7650 4800 50  0001 C CNN
@@
 P 7650 5300
 F 0 "C4" H 7850 5300 50  0000 L CNN
-F 1 "2uf 50V" V 7800 5150 50  0000 L CNN
+F 1 ".2uf 50V" V 7800 5150 50  0000 L CNN
 F 2 "Capacitor_THT:CP_Radial_D6.3mm_P2.50mm" H 7688 5150 50  0001 C CNN
 F 3 "~" H 7650 5300 50  0001 C CNN
@@
 P 8250 5300
 F 0 "C6" H 8250 5150 50  0000 L CNN
-F 1 "1uf 50V" V 8100 5150 50  0000 L CNN
+F 1 ".1uf 50V" V 8100 5150 50  0000 L CNN
 F 2 "Capacitor_THT:CP_Radial_D6.3mm_P2.50mm" H 8288 5150 50  0001 C CNN
 F 3 "~" H 8250 5300 50  0001 C CNN
@@
 Connection ~ 3800 3400
 Text Notes 8750 6800 2    157  ~ 0
-Version V0.1.1
+Version V0.1.2
 $EndSCHEMATC

Commit message: Cap Update
Parts:
- T1: value Myrra 44441 Transformer 240V -> Myrra 44440 Transformer 240V
Changed lines of the file:
@@
 P 5300 5150
 F 0 "T1" H 5300 5731 50  0000 C CNN
-F 1 "Myrra 44441 Transformer 240V " H 5300 5640 50  0000 C CNN
+F 1 "Myrra 44440 Transformer 240V " H 5300 5640 50  0000 C CNN
 F 2 "ROBSLIBRARY:Transformer_Myrra_44440" H 5300 5150 50  0001 C CNN
 F 3 "http://www.farnell.com/datasheets/41284.pdf?_ga=2.233493723.43114568.1597566821-2139994514.1588603417&_gac=1.224077545.1594630648.CjwKCAjwjLD4BRAiEiwAg5NBFqP5waZEob4rUPHshlY-hISIfMy5NeT4Vqv-v37p_oVo35PK2Ko7nhoCuOoQAvD_BwE" H 5300 5150 50  0001 C CNN
